File: led-link/led-link.sch (KiCad schematic (older format))
At the start: 4 parts

Commit message: values
Parts:
- C1: renamed from C?; value C -> 100n; footprint (none) -> Capacitor_SMD:C_0603_1608Metric
- D1: renamed from D?; value 1.5KExxA -> ESDA25P35-1U1M; footprint Diode_THT:D_DO-201AE_P15.24mm_Horizontal -> Diode_SMD:D_0603_1608Metric
- FB1: renamed from FB?; value Ferrite_Bead -> BLM18PG600SZ1D; footprint (none) -> Diode_SMD:D_0603_1608Metric
- gave numbers to parts that had none: 1
Connections:
- net VBUS: now reaches D1.2 (A2), FB1.2, J1.A4 (VBUS), J1.A9 (VBUS), J1.B4 (VBUS), J1.B9 (VBUS)
- net +5V: now reaches C1.1, FB1.1
Changed lines of the file:
@@
 $EndDescr
 $Comp
-L Connector:USB_C_Receptacle_USB2.0 J?
+L Connector:USB_C_Receptacle_USB2.0 J1
 U 1 1 6127DDEF
 P 1750 2400
-F 0 "J?" H 1857 3267 50  0000 C CNN
+F 0 "J1" H 1857 3267 50  0000 C CNN
 F 1 "USB_C_Receptacle_USB2.0" H 1857 3176 50  0000 C CNN
 F 2 "" H 1900 2400 50  0001 C CNN
@@
 NoConn ~ 2350 3000
 $Comp
-L Diode:1.5KExxA D?
+L Diode:1.5KExxA D1
 U 1 1 61283C60
 P 3200 2300
-F 0 "D?" V 3246 2220 50  0000 R CNN
-F 1 "1.5KExxA" V 3155 2220 50  0000 R CNN
-F 2 "Diode_THT:D_DO-201AE_P15.24mm_Horizontal" H 3200 2100 50  0001 C CNN
-F 3 "https://www.vishay.com/docs/88301/15ke.pdf" H 3150 2300 50  0001 C CNN
+F 0 "D1" V 3246 2220 50  0000 R CNN
+F 1 "ESDA25P35-1U1M" V 3155 2220 50  0000 R CNN
+F 2 "Diode_SMD:D_0603_1608Metric" H 3200 2100 50  0001 C CNN
+F 3 "https://www.mouser.es/datasheet/2/389/dm00312034-1798874.pdf" H 3150 2300 50  0001 C CNN
 	1    3200 2300
 	0    -1   -1   0
 $EndComp
 Wire Wire Line
-	2350 1800 3200 1800
+	2350 1800 2900 1800
 Wire Wire Line
 	3200 1800 3200 2150
@@
 	3200 2600 3200 2450
 $Comp
-L Device:Ferrite_Bead FB?
+L Device:Ferrite_Bead FB1
 U 1 1 61286464
 P 3850 1800
-F 0 "FB?" V 3576 1800 50  0000 C CNN
-F 1 "Ferrite_Bead" V 3667 1800 50  0000 C CNN
-F 2 "" V 3780 1800 50  0001 C CNN
-F 3 "~" H 3850 1800 50  0001 C CNN
+F 0 "FB1" V 3576 1800 50  0000 C CNN
+F 1 "BLM18PG600SZ1D" V 3667 1800 50  0000 C CNN
+F 2 "Diode_SMD:D_0603_1608Metric" V 3780 1800 50  0001 C CNN
+F 3 "https://www.mouser.es/datasheet/2/281/QNFA9122-1915769.pdf" H 3850 1800 50  0001 C CNN
 	1    3850 1800
 	0    1    1    0
 $EndComp
 $Comp
-L Device:C C?
+L Device:C C1
 U 1 1 61286FE9
 P 4350 2300
-F 0 "C?" H 4465 2346 50  0000 L CNN
-F 1 "C" H 4465 2255 50  0000 L CNN
-F 2 "" H 4388 2150 50  0001 C CNN
-F 3 "~" H 4350 2300 50  0001 C CNN
+F 0 "C1" H 4465 2346 50  0000 L CNN
+F 1 "100n" H 4465 2255 50  0000 L CNN
+F 2 "Capacitor_SMD:C_0603_1608Metric" H 4388 2150 50  0001 C CNN
+F 3 "https://www.mouser.es/datasheet/2/40/cx5r-776519.pdf" H 4350 2300 50  0001 C CNN
 	1    4350 2300
 	1    0    0    -1
@@
 Wire Wire Line
 	4350 2600 4350 2450
+$Comp
+L power:VBUS #PWR?
+U 1 1 61289DE2
+P 2900 1800
+F 0 "#PWR?" H 2900 1650 50  0001 C CNN
+F 1 "VBUS" H 2915 1973 50  0000 C CNN
+F 2 "" H 2900 1800 50  0001 C CNN
+F 3 "" H 2900 1800 50  0001 C CNN
+	1    2900 1800
+	1    0    0    -1
+$EndComp
+Connection ~ 2900 1800
+Wire Wire Line
+	2900 1800 3200 1800
+$Comp
+L power:+5V #PWR?
+U 1 1 6128A571
+P 4350 1800
+F 0 "#PWR?" H 4350 1650 50  0001 C CNN
+F 1 "+5V" H 4365 1973 50  0000 C CNN
+F 2 "" H 4350 1800 50  0001 C CNN
+F 3 "" H 4350 1800 50  0001 C CNN
+	1    4350 1800
+	1    0    0    -1
+$EndComp
+Connection ~ 4350 1800
 $EndSCHEMATC

Commit message: esp32, alimentacion y power indicator
Parts:
- added C? (x4): 0.1uf, symbol Device:C
- added C? (x4): 1uf, symbol Device:C
- added C?: 10uf, symbol Device:C
- added L?: 2nH, symbol pspice:INDUCTOR
- added R?: 10k, symbol Device:R
- added R?: 82, symbol Device:R
- added SW?: SW_Push, symbol Switch:SW_Push
- added U?: ESP32-PICO-D4, Package_DFN_QFN:QFN-48-1EP_7x7mm_P0.5mm_EP5.3x5.3mm, symbol RF_Module:ESP32-PICO-D4
Connections:
- net labels added: +3.3V, PG, VDDA, VDDA3P3
- wire segments 9 -> 59
Other:
- note added: "Close to ESP32"

Commit message: general changes at schematic
Parts:
- removed U?: ESP32-PICO-D4, Package_DFN_QFN:QFN-48-1EP_7x7mm_P0.5mm_EP5.3x5.3mm, symbol RF_Module:ESP32-PICO-D4
- added A1: PCB Antenna, symbol Connector:Conn_01x02_Female
- added C? (x2): 22pF, symbol Device:C
- added C?: 2.7pF, symbol Device:C
- added C?: 2pF, symbol Device:C
- added C? (x2): C, symbol Device:C
- added D?: LED, symbol Device:LED
- added D?: WS2812B, LED_SMD:LED_WS2812B_PLCC4_5.0x5.0mm_P3.2mm, symbol LED:WS2812B
- added F?: SF-0402F050-2, symbol Device:Fuse
- added L?: 2.7nH, symbol Device:L
- added R?: R0, symbol Device:R
- added R?: 499R, symbol Device:R
- added R?: R, symbol Device:R
- added R? (x2): 5k11, symbol Device:R
- added R?: 1M, symbol Device:R
- added TP?: T_TX, symbol Connector:TestPoint
- added TP?: T_RX, symbol Connector:TestPoint
- added TP?: +5v, symbol Connector:TestPoint
- added TP?: GND, symbol Connector:TestPoint
- added U?: ESP32-PICO-D4, Package_DFN_QFN:QFN-48-1EP_7x7mm_P0.5mm_EP5.3x5.3mm, symbol esp32:ESP32-PICO-D4
- added U?: TPS77633DRG4, symbol led-link:TPS77633DRG4
- added X?: ECS-400-10-36B2-CKM-TR, symbol led-link:ECS-400-10-36B2-CKM-TR
- C? (x4): value 0.1uf -> 0.1uF
- C? (x3): value 1uf -> 1uF
- C?: value 10uf -> 10uF
Connections:
- net labels added: RX, TX, VDD, color_led, status_led
- wire segments 59 -> 132
- no-connect marks 9 -> 7
Other:
- note added: "Color LED"
- note added: "DC Input"
- note added: "LDO"
- note added: "Status"
- note added: "Test"
- moved on the sheet: C1, C?, D1, FB1, J1, L?, R?, SW?

Commit message: push button
Parts:
- added R?: R, symbol Device:R
- added SW?: SW_Push, symbol Switch:SW_Push
Connections:
- net labels added: lna_in, push
- wire segments 132 -> 138
Other:
- note added: "Antena"
- note added: "Push button"
- moved on the sheet: A1, C?, D?, L?, R?, TP?

Commit message: cosas
Parts:
- removed R?: R, symbol Device:R
- removed U?: ESP32-PICO-D4, Package_DFN_QFN:QFN-48-1EP_7x7mm_P0.5mm_EP5.3x5.3mm, symbol esp32:ESP32-PICO-D4
- removed X?: ECS-400-10-36B2-CKM-TR, symbol led-link:ECS-400-10-36B2-CKM-TR
- added C? (x2): C, symbol Device:C
- added R?: R, symbol Device:R
- added U?: ESP32-PICO-D4, Package_DFN_QFN:QFN-48-1EP_7x7mm_P0.5mm_EP5.3x5.3mm, symbol local:ESP32-PICO-D4
- added U?: STM6601CQ2BDM6F, symbol local:STM6601CQ2BDM6F
- added U?: ECS-400-10-36B2-CKM-TR, symbol local:ECS-400-10-36B2-CKM-TR
Connections:
- net labels added: EN_LDO, PB_int, PB_sig, PS_hold
- net labels removed: push
- wire segments 138 -> 160
- no-connect marks 7 -> 10
Other:
- note added: "DNP\nLow ESR"
- note removed: "Push button"
- moved on the sheet: C1, D1, D?, F?, FB1, J1, R?, SW?, TP?

Commit message: more componentts
Parts:
- removed D?: LED, symbol Device:LED
- removed U?: TPS77633DRG4, symbol led-link:TPS77633DRG4
- added C?: 4.7 uF, symbol Device:C
- added D?: HSMF-C169, symbol local:HSMF-C169
- added R? (x2): R, symbol Device:R
- added R?: R0, symbol Device:R
- added U?: MCP73830LT-0AAI, symbol local:MCP73830LT-0AAI
- added U?: TPS77633DRG4, symbol local:TPS77633DRG4
- added U?: BD4737G-TR, symbol local:BD4737G-TR
Connections:
- net labels added: +BATT, charging_led, enable_ldo, hold_power, low_batt, push_button_int, push_button_sig
- net labels removed: EN_LDO, PB_int, PB_sig, PG, PS_hold
- wire segments 160 -> 179
- no-connect marks 10 -> 13
Other:
- moved on the sheet: C?, D?, R?, SW?, U?

Commit message: multiple pages
Parts:
- removed C1: 100n, Capacitor_SMD:C_0603_1608Metric, symbol Device:C
- removed C? (x4): C, symbol Device:C
- removed C?: 4.7 uF, symbol Device:C
- removed D1: ESDA25P35-1U1M, Diode_SMD:D_0603_1608Metric, symbol Diode:1.5KExxA
- removed D?: WS2812B, LED_SMD:LED_WS2812B_PLCC4_5.0x5.0mm_P3.2mm, symbol LED:WS2812B
- removed D?: HSMF-C169, symbol local:HSMF-C169
- removed F?: SF-0402F050-2, symbol Device:Fuse
- removed FB1: BLM18PG600SZ1D, Diode_SMD:D_0603_1608Metric, symbol Device:Ferrite_Bead
- removed J1: USB_C_Receptacle_USB2.0, symbol Connector:USB_C_Receptacle_USB2.0
- removed R?: 499R, symbol Device:R
- removed R? (x4): R, symbol Device:R
- removed R? (x2): 5k11, symbol Device:R
- removed R?: 1M, symbol Device:R
- removed R?: R0, symbol Device:R
- removed SW?: SW_Push, symbol Switch:SW_Push
- removed TP?: +5v, symbol Connector:TestPoint
- removed TP?: GND, symbol Connector:TestPoint
- removed U?: MCP73830LT-0AAI, symbol local:MCP73830LT-0AAI
- removed U?: STM6601CQ2BDM6F, symbol local:STM6601CQ2BDM6F
- removed U?: TPS77633DRG4, symbol local:TPS77633DRG4
- removed U?: BD4737G-TR, symbol local:BD4737G-TR
- gave numbers to parts that had none: 23
Connections:
- net labels removed: +5V, +BATT, RX, TX, VBUS, VDD, charging_led, enable_ldo, hold_power, lna_in, low_batt
- wire segments 179 -> 90
- no-connect marks 13 -> 0
Other:
- note removed: "Antena"
- note removed: "Close to ESP32"
- note removed: "Color LED"
- note removed: "DC Input"
- note removed: "DNP\nLow ESR"
- note removed: "LDO"
- note removed: "Status"
- note removed: "Test"
- moved on the sheet: A1, C1, C10, C11, C12, C13, C2, C3, C4, C5, C6, C7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
